Commit message: mjcf urdf converter

File: robot_sim/urdf/cvrb0609/cvrb0609.urdf (robot description, URDF)
Before this commit: robot model, 34 links, 33 joints
Links:
- link arm1_J1: geometry collision mesh filename=J1.stl scale=1 1 1; visual mesh filename=J1.stl scale=1 1 1
- link arm1_J2: geometry collision mesh filename=J2.stl scale=1 1 1; visual mesh filename=J2.stl scale=1 1 1
- link arm1_J3: geometry collision mesh filename=J3.stl scale=1 1 1; visual mesh filename=J3.stl scale=1 1 1
- link arm1_J4: geometry collision mesh filename=J4.stl scale=1 1 1; visual mesh filename=J4.stl scale=1 1 1
- link arm1_J5: geometry collision mesh filename=J5.stl scale=1 1 1; visual mesh filename=J5.stl scale=1 1 1
- link arm1_J6: geometry collision mesh filename=J6.stl scale=1 1 1; visual mesh filename=J6.stl scale=1 1 1
- link arm1_bottom_link: geometry collision mesh filename=base_link.stl scale=1 1 1; visual mesh filename=base_link.stl scale=1 1 1
- link hand1_robotiq_85_base_link: geometry collision mesh filename=robotiq_arg2f_85_base_link.stl; visual mesh filename=robotiq_arg2f_85_base_link.stl
- link hand1_robotiq_85_left_finger_link: geometry collision mesh filename=robotiq_arg2f_85_outer_finger.stl; visual mesh filename=robotiq_arg2f_85_outer_finger.stl
- link hand1_robotiq_85_left_finger_tip_link: geometry collision mesh filename=robotiq_arg2f_85_inner_finger.stl; visual mesh filename=robotiq_arg2f_85_inner_finger.stl
- link hand1_robotiq_85_left_inner_knuckle_link: geometry collision mesh filename=robotiq_arg2f_85_inner_knuckle.stl; visual mesh filename=robotiq_arg2f_85_inner_knuckle.stl
- link hand1_robotiq_85_left_knuckle_link: geometry collision mesh filename=robotiq_arg2f_85_outer_knuckle.stl; visual mesh filename=robotiq_arg2f_85_outer_knuckle.stl
- link hand1_robotiq_85_right_finger_link: geometry collision mesh filename=robotiq_arg2f_85_outer_finger.stl; visual mesh filename=robotiq_arg2f_85_outer_finger.stl
- link hand1_robotiq_85_right_finger_tip_link: geometry collision mesh filename=robotiq_arg2f_85_inner_finger.stl; visual mesh filename=robotiq_arg2f_85_inner_finger.stl
- link hand1_robotiq_85_right_inner_knuckle_link: geometry collision mesh filename=robotiq_arg2f_85_inner_knuckle.stl; visual mesh filename=robotiq_arg2f_85_inner_knuckle.stl
- link hand1_robotiq_85_right_knuckle_link: geometry collision mesh filename=robotiq_arg2f_85_outer_knuckle.stl; visual mesh filename=robotiq_arg2f_85_outer_knuckle.stl
- link handcover_base_link: geometry collision box size=.1 .1 .1; visual box size=.1 .1 .1
- link robotstand_base_link: geometry collision box size=.1 .1 .1; visual box size=.1 .1 .1
- link robotstand_stage_link: geometry collision box size=.1 .1 .1; visual box size=.1 .1 .1
